File: aerolotl_ab.kicad_pcb (KiCad board)
At the start: 4 copper layers, 152.4 x 152.4 mm, 145 parts, among them J1 FTSH-107-STDC14, J10 GPIO_PE2-PE6, J11 GPIO_PE7-PE11, J12 UART8, J13 SPARE_ADC1, J14 SERVO1, J15 SERVO2, J16 SREVO3, J17 SERVO4, J2 USB_C_Receptacle_USB2.0_16P, J3 Pin Switch Conn, J4 TF-102-15_SD_read, J5 Conn_01x05_Pin, J6 USART3, J7 StemmaQT, J8 StemmaQT, J9 Conn_01x04_Pin, Q1 AO4407A, Q2 AO3400A, SW1 SW_SPST, SW2 SW_Push, U1 STM32H723VGTx, U10 BMP581, U11 Airlift, U2 LMR51430XFDDCR, U3 AMS1117-3.3, U4 USBLC6-2P6, U5 TPS2116DRL, U6 BMI088, U7 ADXL345BCCZ-RL7, U8 MAX-M10S, U9 ADXL375BCCZ-RL7, Y1 X322525MOB4SI, Y2 32k768

Commit message: updated routing and removed extra sensors
Parts:
- removed AE1: GP.1575.18.4.A.02, aerolotl_custom:ANT_GP.1575.18.4.A.02_TAL
- removed C30, C33: 100n, Capacitor_SMD:C_0402_1005Metric
- removed C32: 1u, Capacitor_SMD:C_0402_1005Metric
- removed C34: 10u, Capacitor_SMD:C_0603_1608Metric
- removed FL1: B39162B4300F210, aerolotl_custom:FILTER-SMD_5P-L1.4-W1.1_RSFPXXXXD
- removed R16: 10, Resistor_SMD:R_0402_1005Metric
- removed U7: ADXL345BCCZ-RL7, aerolotl_custom:ADXL345
- removed U8: MAX-M10S, RF_GPS:ublox_MAX
- moved R21 28.7 mm to (153.6, 136.1), turned to 180 degrees
- moved R19 27.6 mm to (153.2, 140.1), turned to 90 degrees
- moved D2 26.0 mm to (156.2, 138.7), turned to 0 degrees
- moved R23 25.8 mm to (154.9, 134.8), turned to 0 degrees
- moved R20 25.1 mm to (153.2, 137.9), turned to 90 degrees
- moved R25 24.9 mm to (163.7, 139.3), turned to -90 degrees
- moved R22 23.1 mm to (154.9, 129.8)
- moved C40 23.1 mm to (169.7, 139.9)
- moved BZ1 22.7 mm to (153.2, 149.3)
- moved D3 22.6 mm to (155.4, 131.3)
- moved Q2 22.6 mm to (166.4, 139.3)
- moved D4 22.5 mm to (155.5, 133.3)
- moved D5 21.8 mm to (158.7, 132.3)
- moved C39 21.1 mm to (165.9, 141.8), turned to 180 degrees
- moved R24 15.8 mm to (160.2, 132.3), turned to 90 degrees
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Connections:
- J1 pad 01: (no net) -> unconnected-(J1-Pad01)
- J1 pad 02: (no net) -> unconnected-(J1-Pad02)
- J1 pad 09: (no net) -> unconnected-(J1-Pad09)
- J1 pad 10: (no net) -> unconnected-(J1-Pad10)
- J2 pad A8: (no net) -> unconnected-(J2-SBU1-PadA8)
- J2 pad B8: (no net) -> unconnected-(J2-SBU2-PadB8)
- U1 pad 17: (no net) -> unconnected-(U1B-PC2_C-Pad17)
- U1 pad 18: (no net) -> unconnected-(U1B-PC3_C-Pad18)
- U1 pad 22: (no net) -> unconnected-(U1B-PA0-Pad22)
- U1 pad 23: (no net) -> unconnected-(U1B-PA1-Pad23)
- U1 pad 24: /Sensors/M10S.RX -> unconnected-(U1B-PA2-Pad24)
- U1 pad 25: /Sensors/M10S.TX -> unconnected-(U1B-PA3-Pad25)
- U1 pad 34: (no net) -> unconnected-(U1B-PB0-Pad34)
- U1 pad 35: (no net) -> unconnected-(U1B-PB1-Pad35)
- U1 pad 61: (no net) -> unconnected-(U1B-PD14-Pad61)
- U1 pad 62: (no net) -> unconnected-(U1B-PD15-Pad62)
- U1 pad 64: /MCU/SPI1.INT_345 -> unconnected-(U1B-PC7-Pad64)
- U1 pad 7: (no net) -> unconnected-(U1B-PC13-Pad7)
- U1 pad 81: (no net) -> unconnected-(U1B-PD0-Pad81)
- U1 pad 87: /MCU/SPI1.CS_345 -> unconnected-(U1B-PD6-Pad87)
- U1 pad 90: (no net) -> unconnected-(U1B-PB4(NJTRST)-Pad90)
- U1 pad 91: /MCU/GPS_RST -> unconnected-(U1B-PB5-Pad91)
- U11 pad 10: (no net) -> unconnected-(U11-GP0-Pad10)
- U11 pad 11: (no net) -> unconnected-(U11-RXI-Pad11)
- U11 pad 12: (no net) -> unconnected-(U11-TXO-Pad12)
- U11 pad 2: (no net) -> unconnected-(U11-3VOut-Pad2)
- U6 pad 1: (no net) -> unconnected-(U6-INT2-Pad1)
- U6 pad 13: (no net) -> unconnected-(U6-INT4-Pad13)
- U9 pad 10: (no net) -> unconnected-(U9-NC-Pad10)
- U9 pad 9: (no net) -> unconnected-(U9-INT2-Pad9)
Routing:
- net /External/GPIO.PE5: track 0.00 -> 116.2 mm, vias 0 -> 4
- net /External/GPIO.PE4: track 0.00 -> 116.0 mm, vias 0 -> 6
- net /MCU/SPI2.BUSY: track 0.00 -> 108.4 mm, vias 0 -> 11
- net /MCU/SPI2.RST: track 0.00 -> 107.7 mm, vias 0 -> 3
- net /External/GPIO.PE7: track 0.00 -> 106.9 mm, vias 0 -> 4
- net /MCU/SPI2.MOSI: track 0.00 -> 106.6 mm, vias 0 -> 1
- net /Power/VOLT_SENSE: track 0.00 -> 104.6 mm, vias 0 -> 4
- net /MCU/SPI2.MISO: track 0.00 -> 103.2 mm, vias 0 -> 4
- net /MCU/SPI2.CS: track 0.00 -> 101.0 mm, vias 0 -> 6
- net /MCU/SPI2.SCK: track 0.00 -> 98.0 mm, vias 0 -> 1
- net /Indicators/LED.G: track 0.00 -> 97.0 mm, vias 0 -> 10
- net /External/GPIO.PE2: track 0.00 -> 95.7 mm, vias 0 -> 6
- net /External/GPIO.PE3: track 0.00 -> 94.0 mm
- net /Debugger/T_NRST: track 0.00 -> 92.0 mm, vias 0 -> 12
- net GND: track 0.00 -> 91.6 mm, vias 0 -> 88
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